Commit message: Fixed reference frame

File: urdf/giraffe.urdf (robot description, URDF)
Before this commit: robot giraffe_robot, 8 links, 7 joints
Joints:
- joint world_joint: origin xyz=0.0 0.0 0.0 rpy=0.0 0.0 0.0 -> xyz=2.5 6.0 4.0 rpy=0.0 0.0 0.0

Commit message: Fixed urdf model with xacro

File: urdf/giraffe.urdf (robot description, URDF)
Before this commit: robot giraffe_robot, 8 links, 7 joints
Links:
- link telescopic_link: geometry collision cylinder length=1.0 radius=0.06; visual cylinder length=1.0 radius=0.06
- link upper_arm_link: geometry collision box size=0.12 0.12 0.8; visual box size=0.12 0.12 0.8
Joints:
- joint telescopic_joint: limit lower=0.0 upper=2.5 effort=200.0 velocity=1.0 -> lower=0.0 upper=6.0 effort=200.0 velocity=1.0; origin xyz=0.0 0.0 -0.15 rpy=0.0 0.0 0.0 -> xyz=0.0 0.0 -0.4 rpy=0.0 0.0 0.0
- joint world_joint: origin xyz=2.5 6.0 4.0 rpy=0.0 0.0 0.0 -> xyz=0.0 0.0 0.0 rpy=0.0 0.0 0.0
- joint wrist_1_joint: origin xyz=0.0 0.0 -0.25 rpy=0.0 0.0 0.0 -> xyz=0.0 0.0 -0.5 rpy=0.0 0.0 0.0

Commit message: Fix urdf

File: urdf/giraffe.urdf (robot description, URDF)
Before this commit: robot giraffe_robot, 8 links, 7 joints
Joints:
- joint world_joint: origin xyz=0.0 0.0 0.0 rpy=0.0 0.0 0.0 -> xyz=2.5 6.0 4.0 rpy=0.0 0.0 0.0

File: urdf/giraffe.urdf.xacro (robot description, xacro)
@@ -1,11 +1,11 @@
 <?xml version="1.0"?>
 <robot name="giraffe_robot" xmlns:xacro="http://www.ros.org/wiki/xacro">
-    <!-- Properties for easy customization -->
+    <!-- Properties -->
     <xacro:property name="PI" value="3.14159265"/>
     <xacro:property name="PI_2" value="1.57079633"/>
-    <!-- Robot mounting position (set to origin for kinematic analysis) -->
-    <xacro:property name="mount_x" value="0.0"/>
-    <xacro:property name="mount_y" value="0.0"/>
-    <xacro:property name="mount_z" value="0.0"/>
+    <!-- Robot mounting position -->
+    <xacro:property name="mount_x" value="2.5"/>
+    <xacro:property name="mount_y" value="6.0"/>
+    <xacro:property name="mount_z" value="4.0"/>
     <!-- Link dimensions -->
     <xacro:property name="base_radius" value="0.1"/>
@@ -27,5 +27,5 @@
     <xacro:property name="base_rotation_limit" value="${PI}"/>
     <xacro:property name="shoulder_tilt_limit" value="${PI_2}"/>
-    <xacro:property name="telescopic_limit" value="6.0"/>
+    <xacro:property name="telescopic_limit" value="6.5"/>
     <xacro:property name="wrist_rotation_limit" value="${PI}"/>
     <xacro:property name="wrist_tilt_limit" value="${PI_2}"/>

Commit message: Last fixes

File: urdf/giraffe.urdf (robot description, URDF)
Before this commit: robot giraffe_robot, 8 links, 7 joints
Joints:
- joint telescopic_joint: limit lower=0.0 upper=6.0 effort=200.0 velocity=1.0 -> lower=0.0 upper=6.5 effort=200.0 velocity=1.0

Commit message: Change wrist max angle

File: urdf/giraffe.urdf (robot description, URDF)
Before this commit: robot giraffe_robot, 8 links, 7 joints
Joints:
- joint wrist_2_joint: limit lower=-1.57079633 upper=1.57079633 effort=50.0 velocity=3.0 -> lower=-2.61799388 upper=2.61799388 effort=50.0 velocity=3.0

File: urdf/giraffe.urdf.xacro (robot description, xacro)
@@ -29,5 +29,5 @@
     <xacro:property name="telescopic_limit" value="6.5"/>
     <xacro:property name="wrist_rotation_limit" value="${PI}"/>
-    <xacro:property name="wrist_tilt_limit" value="${PI_2}"/>
+    <xacro:property name="wrist_tilt_limit" value="${PI} * 5/6"/>
     <!-- Mass properties -->
     <xacro:property name="base_mass" value="5.0"/>
